File: pcb/rotarydial.brd (EAGLE design)
At the start: 42.9 x 61 mm, 44 parts, among them IC1 TINY85V, IC2 L78L05, J1 J5MM, J2 J5MM, J3 J15MM, J4 J10MM, J5 J20MM, J6 J5MM, J7 J5MM, K2 TX2-L2-3V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

Commit message: Fixed some design errors of board rev. A. This is now officially board rev. B.
Parts:
- removed K3: TX2-L2-3V, relay:TX2-L2
- added J8: J5MM, jumper:05
- added K1: EC2-3TNU, relay-custom:TX2-L2
- J1: value J5MM -> J10MM; device jumper:05 -> jumper:10
- K2: value TX2-L2-3V -> EC2-3TNU; device relay:TX2-L2 -> relay-custom:TX2-L2
- R3, R4: value 680 -> 470
- T1, T2: device triac:TO92-4 -> triac:TO92-2
- moved K2 12.1 mm to (19.1, 55.9), turned to 180 degrees
- moved J1 7.33 mm to (16.8, 38.4), turned to 180 degrees
- moved T2 1.27 mm to (29.5, 44.8), turned to 0 degrees
- moved PPLS 1.27 mm to (21.6, 49.5)
- moved T1 1.27 mm to (29.5, 58.1), turned to 90 degrees
- moved D7 1.00 mm to (29.8, 37.5)
- moved R4 0.90 mm to (33.7, 41.3)
- turned D4 to 90 degrees
- turned D5 to 90 degrees
Connections:
- removed net N$12: D9.A, K2.12, S1.1
- removed net N$27: J3.2, K3.7
- new net N$16: J8.1, K1.7
- new net N$17: D9.A, J8.2, S1.1
- new net N$7: J3.2, K2.6
- net GND: now also D4.A, D5.A, K1.5; no longer D4.C, D5.C, K2.5
- net N$1: now also D5.C; no longer D5.A
- net N$10: now also K2.9; no longer K3.9
- net N$11: now also K1.6; no longer K3.12
- net N$15: now also K2.5; no longer K3.5
- net N$18: now also K1.9; no longer K2.9
- net N$2: now also D4.C; no longer D4.A
- net N$20: now also K1.4; no longer K2.4
- net N$28: now also K2.8; no longer K3.8
- net N$4: now also K2.3; no longer K3.3
- net N$5: now also K1.1, K2.12; no longer K2.1, K3.6
- net N$6: now also K1.12; no longer K2.6
- net N$8: now also K2.1; no longer K3.1
- net PCOM: now also K1.3; no longer K2.3
- net PMTE: now also K1.10; no longer K2.10
- net PPLS: now also K2.10; no longer K3.10
- net R2: now also K2.4; no longer K3.4
- net R_DIAL_MUTE: now also K1.8; no longer K2.8
Routing:
- net N$12: track 37.9 -> 0.00 mm
- net N$11: track 6.99 -> 42.9 mm
- net N$5: track 24.7 -> 47.8 mm
- net N$17: track 0.00 -> 15.8 mm
- net N$16: track 0.00 -> 9.78 mm
- net N$7: track 0.00 -> 7.77 mm
- net N$6: track 3.72 -> 10.3 mm
- net N$25: track 2.01 -> 5.53 mm
- net N$24: track 2.04 -> 4.58 mm
- net N$27: track 2.01 -> 0.00 mm
- net N$8: track 47.5 -> 49.1 mm
- net N$15: track 34.3 -> 35.8 mm
- net N$28: track 18.7 -> 17.3 mm
- net PPLS: track 29.3 -> 28.0 mm
- net N$26: track 22.0 -> 23.2 mm
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Other:
- board size 42.9 x 61 mm -> 42.9 x 61.9 mm
- board text added: "PULSE-TONE ROTARY DIAL rev. B, 2024"
- board text removed: "PULSE-TONE ROTARY DIAL rev. A, 2024"
