File: pcb/rotarydial.sch (EAGLE design)
At the start: 44 parts, among them IC1 TINY85V, IC2 L78L05, J1 J5MM, J2 J5MM, J3 J15MM, J4 J10MM, J5 J20MM, J6 J5MM, J7 J5MM, K2 TX2-L2-3V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

Commit message: Fixed some design errors of board rev. A. This is now officially board rev. B.
Parts:
- removed K3: TX2-L2-3V, relay:TX2-L2-3V
- added J8: J5MM, jumper:J5MM
- added K1: EC2-3TNU, relay-custom:TX2LT-L2-
- J1: value J5MM -> J10MM; device jumper:J5MM -> jumper:J10MM
- K2: value TX2-L2-3V -> EC2-3TNU; device relay:TX2-L2-3V -> relay-custom:TX2LT-L2-
- R3, R4: value 680 -> 470
- T1, T2: device triac:BT149 -> triac:BT169
Connections:
- removed net N$12: D9.A, K2S.+, S11.S
- removed net N$27: J3.2, K3S.-
- new net N$16: J8.1, K1S.-
- new net N$17: D9.A, J8.2, S11.S
- new net N$7: J3.2, K2S.+
- net GND: now also D4.A, D5.A, K11.S; no longer D4.C, D5.C, K21.S
- net N$1: now also D5.C; no longer D5.A
- net N$10: now also K22.P; no longer K32.P
- net N$11: now also K1S.+; no longer K3S.+
- net N$15: now also K21.S; no longer K31.S
- net N$18: now also K12.P; no longer K22.P
- net N$2: now also D4.C; no longer D4.A
- net N$20: now also K11.P; no longer K21.P
- net N$28: now also K22.S; no longer K32.S
- net N$4: now also K21.O; no longer K31.O
- net N$5: now also K1R.+, K2R.-; no longer K2R.+, K3R.-
- net N$6: now also K1R.-; no longer K2R.-
- net N$8: now also K2R.+; no longer K3R.+
- net PCOM: now also K11.O; no longer K21.O
- net PMTE: now also K12.O; no longer K22.O
- net PPLS: now also K22.O; no longer K32.O
- net R2: now also K21.P; no longer K31.P
- net R_DIAL_MUTE: now also K12.S; no longer K22.S
Other:
- moved on the sheet: D4, D5, D6, K2, T1
